Commit message: setup

File: src/pkg_binx/description/binx.urdf.xacro (robot description, xacro)
@@ -1,4 +1,4 @@
 <?xml version="1.0"?>
-<robot xmlns:xacro="http://www.ros.org/wiki/xacro" name="binx">
-    <link name = "base_link"></link>
+<robot xmlns:xacro="http://www.ros.org/wiki/xacro" name="robot">
+    <xacro:include filename="binx_core.xacro" />
 </robot>

Commit message: gazebo works!!

File: src/pkg_binx/description/binx.urdf.xacro (robot description, xacro)
@@ -1,4 +1,4 @@
 <?xml version="1.0"?>
-<robot xmlns:xacro="http://www.ros.org/wiki/xacro" name="robot">
+<robot xmlns:xacro="http://www.ros.org/wiki/xacro" name="binx">
     <xacro:include filename="binx_core.xacro" />
 </robot>

File: src/pkg_binx/description/binx_core.xacro (robot description, xacro)
@@ -1,32 +1,199 @@
 <?xml version="1.0"?>
 <robot xmlns:xacro="http://www.ros.org/wiki/xacro" >
+    <!-- *remember to cite and ref aleksander haber btw* -->
+    <!-- ########################## -->
+    <!-- Including additional files -->
+    <!-- ########################## -->
+    <!-- <xacro:include filename = "${find pkg_binx}/description/robot.gazebo" /> -->
+    <!-- ######################## -->
+    <!-- Defining robot constants -->
+    <!-- ######################## -->
+    <xacro:property name = "pi_const" value = "3.14159265" />
+    <!-- colors -->
     <material name="white">
         <color rgba="1 1 1 1" />
     </material>
-    <material name="orange">
-        <color rgba="1 0.3 0.1 1"/>
+    <material name="blue">
+        <color rgba="0.150 0.178 0.242 1"/>
     </material>
-    <material name="blue">
-        <color rgba="0.2 0.2 1 1"/>
+    <material name="pink">
+        <color rgba="0.237 0.199 0.220 1"/>
     </material>
     <material name="black">
         <color rgba="0 0 0 1"/>
     </material>
-    <!-- BASE LINK -->
-    <link name="base_link">
+    <!-- chassis dimensions -->
+    <xacro:property name = "l" value = "1" />
+    <xacro:property name = "h" value = "0.3" />
+    <xacro:property name = "w" value = "0.75" />
+    <!-- wheel radius and diameter -->
+    <xacro:property name = "r" value = "0.15" />
+    <xacro:property name = "d" value = "0.1" />
+    <!-- other dimensions (look at aleks' vid for the full picture)-->
+    <xacro:property name = "s1" value = "${h/2 + r}" />
+    <xacro:property name = "s2" value = "${2*r}" />
+    <xacro:property name = "s3" value = "${2*r}" />
+    <xacro:property name = "s4" value = "${w/2 + d/2}" />
+    <!-- ##################################### -->
+    <!-- Defining mass and inertial properites -->
+    <!-- ##################################### -->
+    <!-- material densities -->
+    <xacro:property name = "bodyDensity" value = "2710.0" />
+    <xacro:property name = "wheelDensity" value = "2710.0" />
+    <!-- mass -->
+    <xacro:property name = "bodyMass" value = "${bodyDensity*l*h*w}" />
+    <xacro:property name = "wheelMass" value = "${wheelDensity*pi_const*r*r*d}" />
+    <!-- moments of inertia -->
+    <xacro:property name = "Ix_body" value = "${(1/12)*bodyMass*(h*h + w*w)}" />
+    <xacro:property name = "Iy_body" value = "${(1/12)*bodyMass*(l*l + h*h)}" />
+    <xacro:property name = "Iz_body" value = "${(1/12)*bodyMass*(l*l + w*w)}" />
+    <xacro:property name = "Iz_wheel" value = "${0.5*wheelMass*r*r}" />
+    <xacro:property name = "I_wheel" value = "${(1.0/12.0)*wheelMass*(3.0*r*r + d*d)}" />
+    <!-- inertial macros -->
+    <xacro:macro name = "inertia_body">
+        <inertial>
+            <origin rpy = "0 0 0" xyz = "0 0 ${s1}" />
+            <mass value = "${bodyMass}" />
+            <inertia ixx = "${Ix_body}" ixy = "0.0" ixz = "0.0" iyy = "${Iy_body}" iyz = "0" izz = "${Iz_body}" />
+        </inertial>
+    </xacro:macro>
+    <xacro:macro name = "inertia_wheel">
+        <inertial>
+            <origin rpy = "1.570795 0 0" xyz = "0 0 0" />
+            <mass value = "${wheelMass}" />
+            <inertia ixx = "${I_wheel}" ixy = "0.0" ixz = "0.0" iyy = "${I_wheel}" iyz = "0" izz = "${Iz_wheel}" />
+        </inertial>
+    </xacro:macro>
+    <!-- ####################### -->
+    <!-- Defining links & joints -->
+    <!-- ####################### -->
+    <!-- ficitous link -->
+    <link name = "base_footprint"> </link>
+    <joint name = "body_link_joint" type = "fixed">
+        <parent link = "base_footprint" />
+        <child link = "body_link" />
+    </joint>
+    <!-- body link -->
+    <!-- *figure out if you need to change the origin's x value to -0.1 or sum* -->
+    <!-- *also idk if you need to add the color to the collision asw prolly not* -->
+    <link name = "body_link">
+        <visual>
+            <origin rpy = "0 0 0" xyz = "0 0 ${s1}" />
+            <geometry>
+                <box size = "${l} ${w} ${h}" />
+            </geometry>
+            <material name = "blue" />
+        </visual>
+        <collision>
+            <origin rpy = "0 0 0" xyz = "0 0 ${s1}" />
+            <geometry>
+                <box size = "${l} ${w} ${h}" />
+            </geometry>
+        </collision>
+        <xacro:inertia_body />
     </link>
-    <joint name="chassis_joint" type="fixed">
-        <parent link = "base_link" />
-        <child link = "chassis" />
-        <origin xyz= "-0.1 0 0"/>
+    <!-- right wheel rear link -->
+    <!-- remember to make the limit effort more realistic later... -->
+    <joint name= "wheel1_joint" type = "continuous">
+        <parent link = "body_link" />
+        <child link = "wheel1_link" />
+        <origin xyz = "${-s2} ${-s4} ${r}" rpy = "0 0 0" />
+        <axis xyz = "0 1 0" />
+        <limit effort = "50000" velocity = "10" />
+        <dynamics damping = "1.0" friction = "1.0" />
     </joint>
-    <link name="chassis">
+    <link name = "wheel1_link">
         <visual>
-            <origin xyz="0.15 0 0.075"/>
+            <origin rpy = "1.570795 0 0" xyz = "0 0 0" />
             <geometry>
-                <box size="0.3 0.3 0.15"/>
+                <cylinder length = "${d}" radius = "${r}" />
             </geometry>
-            <material name="white"/>
+            <material name = "pink" />
         </visual>
+        <collision>
+            <origin rpy = "1.57095 0 0" xyz = "0 0 0" />
+            <geometry>
+                <cylinder length = "${d}" radius = "${r}" />
+            </geometry>
+        </collision>
+        <xacro:inertia_wheel />
+    </link>
+    <!-- left wheel rear link -->
+    <!-- remember to make the limit effort more realistic later... -->
+    <joint name= "wheel2_joint" type = "continuous">
+        <parent link = "body_link" />
+        <child link = "wheel2_link" />
+        <origin xyz = "${-s2} ${s4} ${r}" rpy = "0 0 0" />
+        <axis xyz = "0 1 0" />
+        <limit effort = "50000" velocity = "10" />
+        <dynamics damping = "1.0" friction = "1.0" />
+    </joint>
+    <link name = "wheel2_link">
+        <visual>
+            <origin rpy = "1.570795 0 0" xyz = "0 0 0" />
+            <geometry>
+                <cylinder length = "${d}" radius = "${r}" />
+            </geometry>
+            <material name = "pink" />
+        </visual>
+        <collision>
+            <origin rpy = "1.57095 0 0" xyz = "0 0 0" />
+            <geometry>
+                <cylinder length = "${d}" radius = "${r}" />
+            </geometry>
+        </collision>
+        <xacro:inertia_wheel />
+    </link>
+    <!-- right wheel forward link -->
+    <!-- remember to make the limit effort more realistic later... -->
+    <joint name= "wheel3_joint" type = "continuous">
+        <parent link = "body_link" />
+        <child link = "wheel3_link" />
+        <origin xyz = "${s2} ${-s4} ${r}" rpy = "0 0 0" />
+        <axis xyz = "0 1 0" />
+        <limit effort = "50000" velocity = "10" />
+        <dynamics damping = "1.0" friction = "1.0" />
+    </joint>
+    <link name = "wheel3_link">
+        <visual>
+            <origin rpy = "1.570795 0 0" xyz = "0 0 0" />
+            <geometry>
+                <cylinder length = "${d}" radius = "${r}" />
+            </geometry>
+            <material name = "pink" />
+        </visual>
+        <collision>
+            <origin rpy = "1.57095 0 0" xyz = "0 0 0" />
+            <geometry>
+                <cylinder length = "${d}" radius = "${r}" />
+            </geometry>
+        </collision>
+        <xacro:inertia_wheel />
+    </link>
+    <!-- left wheel forward link -->
+    <!-- remember to make the limit effort more realistic later... -->
+    <joint name= "wheel4_joint" type = "continuous">
+        <parent link = "body_link" />
+        <child link = "wheel4_link" />
+        <origin xyz = "${s2} ${s4} ${r}" rpy = "0 0 0" />
+        <axis xyz = "0 1 0" />
+        <limit effort = "50000" velocity = "10" />
+        <dynamics damping = "1.0" friction = "1.0" />
+    </joint>
+    <link name = "wheel4_link">
+        <visual>
+            <origin rpy = "1.570795 0 0" xyz = "0 0 0" />
+            <geometry>
+                <cylinder length = "${d}" radius = "${r}" />
+            </geometry>
+            <material name = "pink" />
+        </visual>
+        <collision>
+            <origin rpy = "1.57095 0 0" xyz = "0 0 0" />
+            <geometry>
+                <cylinder length = "${d}" radius = "${r}" />
+            </geometry>
+        </collision>
+        <xacro:inertia_wheel />
     </link>
 </robot>

Commit message: changes with mecanum added

File: src/pkg_binx/description/binx.urdf.xacro (robot description, xacro)
@@ -2,3 +2,4 @@
 <robot xmlns:xacro="http://www.ros.org/wiki/xacro" name="binx">
     <xacro:include filename="binx_core.xacro" />
+    <xacro:include filename="lidar.xacro" />
 </robot>

File: src/pkg_binx/description/binx_core.xacro (robot description, xacro)
@@ -2,25 +2,21 @@
 <robot xmlns:xacro="http://www.ros.org/wiki/xacro" >
     <!-- *remember to cite and ref aleksander haber btw* -->
-    <!-- ########################## -->
-    <!-- Including additional files -->
-    <!-- ########################## -->
-    <!-- <xacro:include filename = "${find pkg_binx}/description/robot.gazebo" /> -->
+    <!-- colors -->
+    <material name="white">
+        <color rgba="1 1 1 1" />
+    </material>
+    <material name="blue">
+        <color rgba="0.150 0.178 0.242 1"/>
+    </material>
+    <material name="pink">
+        <color rgba="0.237 0.199 0.220 1"/>
+    </material>
+    <material name="black">
+        <color rgba="0 0 0 1"/>
+    </material>
     <!-- ######################## -->
     <!-- Defining robot constants -->
     <!-- ######################## -->
     <xacro:property name = "pi_const" value = "3.14159265" />
-    <!-- colors -->
-    <material name="white">
-        <color rgba="1 1 1 1" />
-    </material>
-    <material name="blue">
-        <color rgba="0.150 0.178 0.242 1"/>
-    </material>
-    <material name="pink">
-        <color rgba="0.237 0.199 0.220 1"/>
-    </material>
-    <material name="black">
-        <color rgba="0 0 0 1"/>
-    </material>
     <!-- chassis dimensions -->
     <xacro:property name = "l" value = "1" />
@@ -68,6 +64,8 @@
     <!-- Defining links & joints -->
     <!-- ####################### -->
-    <!-- ficitous link -->
-    <link name = "base_footprint"> </link>
+    <!-- fictitious link -->
+    <link name = "base_footprint">
+        <xacro:inertia_body />
+    </link>
     <joint name = "body_link_joint" type = "fixed">
         <parent link = "base_footprint" />
@@ -76,5 +74,4 @@
     <!-- body link -->
     <!-- *figure out if you need to change the origin's x value to -0.1 or sum* -->
-    <!-- *also idk if you need to add the color to the collision asw prolly not* -->
     <link name = "body_link">
         <visual>
@@ -197,3 +194,7 @@
         <xacro:inertia_wheel />
     </link>
+    <!-- ########################## -->
+    <!-- Including additional files -->
+    <!-- ########################## -->
+    <xacro:include filename = "$(find pkg_binx)/description/robot.gazebo" />
 </robot>

Commit message: lidar+cam

File: src/pkg_binx/description/binx.urdf.xacro (robot description, xacro)
@@ -3,3 +3,4 @@
     <xacro:include filename="binx_core.xacro" />
     <xacro:include filename="lidar.xacro" />
+    <xacro:include filename="camera.xacro" />
 </robot>

File: src/pkg_binx/description/binx_core.xacro (robot description, xacro)
@@ -66,5 +66,4 @@
     <!-- fictitious link -->
     <link name = "base_footprint">
-        <xacro:inertia_body />
     </link>
     <joint name = "body_link_joint" type = "fixed">

File: src/pkg_binx/description/lidar.xacro (robot description, xacro)
@@ -1,8 +1,8 @@
 <?xml version ="1.0"?>
-<robot xmlns:xacro = "https://www.ros.org/wiki/xacro">
+<robot xmlns:xacro = "http://www.ros.org/wiki/xacro">
     <joint name = "lidar_joint" type = "fixed">
         <parent link = "body_link"/>
         <child link = "lidar_link"/>
-        <origin xyz = "0 0 ${h/2 + 0.05}" rpy = "0 0 0"/>
+        <origin xyz = "0 0 ${s1 + h/2 + 0.05}" rpy = "0 0 0"/>
     </joint>
     <link name = "lidar_link">
@@ -17,5 +17,5 @@
         </visual>
         <collision>
-            <origin xyz = "0 0 0.05" rpy = "0 0 0"/>
+            <origin xyz = "0 0 0" rpy = "0 0 0"/>
             <geometry>
                 <cylinder radius = "0.03" length = "0.1"/>
