Commit message: Added line-following-color-detection environment (read launch file)

File: src/pkg_binx/description/binx_core.xacro (robot description, xacro)
@@ -61,4 +61,8 @@
         </inertial>
     </xacro:macro>
+    <!-- ########################## -->
+    <!-- Including additional files -->
+    <!-- ########################## -->
+    <xacro:include filename = "$(find pkg_binx)/description/robot.gazebo" />
     <!-- ####################### -->
     <!-- Defining links & joints -->
@@ -108,9 +112,18 @@
             <material name = "pink" />
         </visual>
-        <collision>
-            <origin rpy = "1.57095 0 0" xyz = "0 0 0" />
-            <geometry>
-                <cylinder length = "${d}" radius = "${r}" />
-            </geometry>
+        <collision name = "wheel1_collision">
+            <origin rpy = "1.57095 0 0" xyz = "0 0 0" />
+            <geometry>
+                <cylinder length = "${d}" radius = "${r}" />
+            </geometry>
+            <surface>
+                <friction>
+                    <ode>
+                        <mu>2.0</mu>
+                        <mu2>0.01</mu2>
+                        <fdir1>-1 -1 0</fdir1>
+                    </ode>
+                </friction>
+            </surface>
         </collision>
         <xacro:inertia_wheel />
@@ -134,9 +147,18 @@
             <material name = "pink" />
         </visual>
-        <collision>
-            <origin rpy = "1.57095 0 0" xyz = "0 0 0" />
-            <geometry>
-                <cylinder length = "${d}" radius = "${r}" />
-            </geometry>
+        <collision name = "wheel2_collision">
+            <origin rpy = "1.57095 0 0" xyz = "0 0 0" />
+            <geometry>
+                <cylinder length = "${d}" radius = "${r}" />
+            </geometry>
+            <surface>
+                <friction>
+                    <ode>
+                        <mu>2.0</mu>
+                        <mu2>0.01</mu2>
+                        <fdir1>-1 1 0</fdir1>
+                    </ode>
+                </friction>
+            </surface>
         </collision>
         <xacro:inertia_wheel />
@@ -160,9 +182,18 @@
             <material name = "pink" />
         </visual>
-        <collision>
-            <origin rpy = "1.57095 0 0" xyz = "0 0 0" />
-            <geometry>
-                <cylinder length = "${d}" radius = "${r}" />
-            </geometry>
+        <collision name = "wheel3_collision">
+            <origin rpy = "1.57095 0 0" xyz = "0 0 0" />
+            <geometry>
+                <cylinder length = "${d}" radius = "${r}" />
+            </geometry>
+            <surface>
+                <friction>
+                    <ode>
+                        <mu>2.0</mu>
+                        <mu2>0.01</mu2>
+                        <fdir1>1 -1 0</fdir1>
+                    </ode>
+                </friction>
+            </surface>
         </collision>
         <xacro:inertia_wheel />
@@ -186,15 +217,20 @@
             <material name = "pink" />
         </visual>
-        <collision>
-            <origin rpy = "1.57095 0 0" xyz = "0 0 0" />
-            <geometry>
-                <cylinder length = "${d}" radius = "${r}" />
-            </geometry>
-        </collision>
-        <xacro:inertia_wheel />
-    </link>
-    <!-- ########################## -->
-    <!-- Including additional files -->
-    <!-- ########################## -->
-    <xacro:include filename = "$(find pkg_binx)/description/robot.gazebo" />
+        <collision name = "wheel4_collision">
+            <origin rpy = "1.57095 0 0" xyz = "0 0 0" />
+            <geometry>
+                <cylinder length = "${d}" radius = "${r}" />
+            </geometry>
+            <surface>
+                <friction>
+                    <ode>
+                        <mu>2.0</mu>
+                        <mu2>0.01</mu2>
+                        <fdir1>1 1 0</fdir1>
+                    </ode>
+                </friction>
+            </surface>
+        </collision>
+        <xacro:inertia_wheel />
+    </link>
 </robot>

File: src/pkg_binx/description/lidar.xacro (robot description, xacro)
@@ -1,8 +1,8 @@
 <?xml version ="1.0"?>
-<robot xmlns:xacro = "https://www.ros.org/wiki/xacro">
+<robot xmlns:xacro = "http://www.ros.org/wiki/xacro">
     <joint name = "lidar_joint" type = "fixed">
         <parent link = "body_link"/>
         <child link = "lidar_link"/>
-        <origin xyz = "0 0 ${h/2 + 0.05}" rpy = "0 0 0"/>
+        <origin xyz = "0 0 ${s1 + h/2 + 0.05}" rpy = "0 0 0"/>
     </joint>
     <link name = "lidar_link">
@@ -17,5 +17,5 @@
         </visual>
         <collision>
-            <origin xyz = "0 0 0.05" rpy = "0 0 0"/>
+            <origin xyz = "0 0 0" rpy = "0 0 0"/>
             <geometry>
                 <cylinder radius = "0.03" length = "0.1"/>

Commit message: working line follower

File: src/pkg_binx/description/binx_core.xacro (robot description, xacro)
@@ -15,16 +15,21 @@
         <color rgba="0 0 0 1"/>
     </material>
+    <material name = "gray">
+        <color rgba = "0.05 0.05 0.05 1"/>
+    </material>
     <!-- ######################## -->
     <!-- Defining robot constants -->
     <!-- ######################## -->
     <xacro:property name = "pi_const" value = "3.14159265" />
+    <!-- modifier -->
+    <xacro:property name = "m" value = "1" />
     <!-- chassis dimensions -->
-    <xacro:property name = "l" value = "1" />
-    <xacro:property name = "h" value = "0.3" />
-    <xacro:property name = "w" value = "0.75" />
+    <xacro:property name = "l" value = "${m*1}" />
+    <xacro:property name = "h" value = "${m*0.3}" />
+    <xacro:property name = "w" value = "${m*0.75}" />
     <!-- wheel radius and diameter -->
-    <xacro:property name = "r" value = "0.15" />
-    <xacro:property name = "d" value = "0.1" />
-    <!-- other dimensions (look at aleks' vid for the full picture)-->
+    <xacro:property name = "r" value = "${m*0.15}" />
+    <xacro:property name = "d" value = "${m*0.1}" />
+    <!-- other dimensions (look at aleks's vid for the full picture)-->
     <xacro:property name = "s1" value = "${h/2 + r}" />
     <xacro:property name = "s2" value = "${2*r}" />

File: src/pkg_binx/description/camera.xacro (robot description, xacro)
@@ -2,5 +2,5 @@
 <robot xmlns:xacro="http://www.ros.org/wiki/xacro" >
     <joint type="fixed" name="camera_joint">
-        <origin xyz="0.5 0 0.3" rpy="0 0 0"/>
+        <origin xyz="${l/2} 0 ${h}" rpy="0 0 0"/>
         <child link="camera_link"/>
         <parent link="body_link"/>
@@ -29,4 +29,5 @@
                 <box size=".03 .03 .03"/>
             </geometry>
+            <material name = "gray" />
         </visual>
     </link>
@@ -38,25 +39,3 @@
     <link name="camera_link_optical">
     </link>
-    <gazebo reference="camera_link">
-        <material>Gazebo/Red</material>
-        <sensor name="camera" type="camera">
-            <pose> 0 0 0 0 0 0 </pose>
-            <visualize>true</visualize>
-            <update_rate>20</update_rate>
-            <topic>camera/image</topic>
-            <gz_frame_id>camera_link_optical</gz_frame_id>
-            <camera>
-                <horizontal_fov>1.3962634</horizontal_fov>
-                <image>
-                    <format>R8G8B8</format>
-                    <width>640</width>
-                    <height>480</height>
-                </image>
-                <clip>
-                    <near>0.1</near>
-                    <far>15</far>
-                </clip>
-            </camera>
-        </sensor>
-    </gazebo>
 </robot>

File: src/pkg_binx/description/lidar.xacro (robot description, xacro)
@@ -10,14 +10,12 @@
             <origin xyz = "0 0 0" rpy = "0 0 0"/>
             <geometry>
-                <cylinder radius = "0.03" length = "0.1"/>
+                <cylinder radius = "${d}" length = "${d}"/>
             </geometry>
-            <material name = "black">
-                <color rgba = "0 0 0 1"/>
-            </material>
+            <material name = "gray" />
         </visual>
         <collision>
             <origin xyz = "0 0 0" rpy = "0 0 0"/>
             <geometry>
-                <cylinder radius = "0.03" length = "0.1"/>
+                <cylinder radius = "${d}" length = "${d}"/>
             </geometry>
         </collision>
